File: hardware/motor-pid-ctrl/robot-power.sch (KiCad schematic (older format))
At the start: 49 parts, among them IC1 ATMEGA328-P, IC2 L6202, M1 MOTOR, P1 MAINS, P2 AVR ISP, P3 IO PORTS, Q1 BP103, T1 30VA, T2 1VA, X1 18.432Mhz

Commit message: Adjustments. Starting to lay trackings
Parts:
- renumbered LR1 to IC4
Connections:
- net at R16.2, SSR1.4 (S2), T2.2 (AB): no longer R2.1
- net at P1.2 (PM), R16.1, T1.1 (IN+)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: now also R2.1
